File: pan-mix.kicad_sch (KiCad schematic)
At the start: 296 parts

Commit message: changing audio jacks
Parts:
- removed J?: CV 1, symbol Connector:AudioJack2
- removed J?: IN 3, symbol Connector:AudioJack2
- removed J?: CV 4, symbol Connector:AudioJack2
- removed J?: CV 3, symbol Connector:AudioJack2
- removed J?: IN 4, symbol Connector:AudioJack2
- removed J?: IN 1, symbol Connector:AudioJack2
- removed J?: CV 2, symbol Connector:AudioJack2
- removed J?: IN 2, symbol Connector:AudioJack2
- added J?: CV 4, symbol Connector:AudioJack2_SwitchT
- added J?: CV 3, symbol Connector:AudioJack2_SwitchT
- added J?: IN 4, symbol Connector:AudioJack2_SwitchT
- added J?: IN 2, symbol Connector:AudioJack2_SwitchT
- added J?: CV 2, symbol Connector:AudioJack2_SwitchT
- added J?: IN 1, symbol Connector:AudioJack2_SwitchT
- added J?: CV 1, symbol Connector:AudioJack2_SwitchT
- added J?: IN 3, symbol Connector:AudioJack2_SwitchT
Connections:
- net GND: now also J?.S, J?.S, J?.S, J?.S, J?.S, J?.S, J?.S, J?.S
- net at RV?.3: now also J?.T (x8)
- no-connect marks 0 -> 8

Commit message: some footprints
Parts:
- removed J? (x3): Conn_02x04_Odd_Even, symbol Connector_Generic:Conn_02x04_Odd_Even
- added H1: lvl 1, Eurorack:Mech-Potentiometer-Hole_level, symbol Mechanical:MountingHole
- added H10: in 2, Eurorack:Mech-AudioJack-Hole, symbol Mechanical:MountingHole
- added H11: lvl 3, Eurorack:Mech-Potentiometer-Hole_level, symbol Mechanical:MountingHole
- added H12: pan 3, Eurorack:Mech-Potentiometer-Hole_pan, symbol Mechanical:MountingHole
- added H13: cv 3, Eurorack:Mech-Potentiometer-Hole_level, symbol Mechanical:MountingHole
- added H14: cv 3, Eurorack:Mech-AudioJack-Hole, symbol Mechanical:MountingHole
- added H15: in 3, Eurorack:Mech-AudioJack-Hole, symbol Mechanical:MountingHole
- added H16: lvl4, Eurorack:Mech-Potentiometer-Hole_level, symbol Mechanical:MountingHole
- added H17: pan 4, Eurorack:Mech-Potentiometer-Hole_pan, symbol Mechanical:MountingHole
- added H18: cv 4, Eurorack:Mech-Potentiometer-Hole_level, symbol Mechanical:MountingHole
- added H19: cv 4, Eurorack:Mech-AudioJack-Hole, symbol Mechanical:MountingHole
- added H2: pan 1, Eurorack:Mech-Potentiometer-Hole_pan, symbol Mechanical:MountingHole
- added H20: in 4, Eurorack:Mech-AudioJack-Hole, symbol Mechanical:MountingHole
- added H21: main lvl, Eurorack:Mech-Potentiometer-Hole_level, symbol Mechanical:MountingHole
- added H22: treble, Eurorack:Mech-Potentiometer-Hole_pan, symbol Mechanical:MountingHole
- added H23: bass, Eurorack:Mech-Potentiometer-Hole_pan, symbol Mechanical:MountingHole
- added H24: left, Eurorack:Mech-AudioJack-Hole, symbol Mechanical:MountingHole
- added H25: right, Eurorack:Mech-AudioJack-Hole, symbol Mechanical:MountingHole
- added H26: phones, Eurorack:Mech-AudioJack-Hole-0_25-L12B, symbol Mechanical:MountingHole
- added H27: phones lvl, Eurorack:Mech-AudioJack-Hole-0_25-L12B, symbol Mechanical:MountingHole
- added H3: cv 1, Eurorack:Mech-Potentiometer-Hole_level, symbol Mechanical:MountingHole
- added H4: cv 1, Eurorack:Mech-AudioJack-Hole, symbol Mechanical:MountingHole
- added H5: in 1, Eurorack:Mech-AudioJack-Hole, symbol Mechanical:MountingHole
- added H6: lvl 2, Eurorack:Mech-Potentiometer-Hole_level, symbol Mechanical:MountingHole
- added H7: pan 2, Eurorack:Mech-Potentiometer-Hole_pan, symbol Mechanical:MountingHole
- added H8: cv 2, Eurorack:Mech-Potentiometer-Hole_level, symbol Mechanical:MountingHole
- added H9: cv 2, Eurorack:Mech-AudioJack-Hole, symbol Mechanical:MountingHole
- added J19: left, Eurorack:AudioJack2_Tayda_A-2566, symbol Connector:AudioJack2_SwitchT
- added J20, J22: Conn_01x03_Female, Connector_PinSocket_2.54mm:PinSocket_1x03_P2.54mm_Vertical, symbol Connector:Conn_01x03_Female
- added J21: right, Eurorack:AudioJack2_Tayda_A-2566, symbol Connector:AudioJack2_SwitchT
- added J23: Conn_02x05_Odd_Even, Connector_PinHeader_2.54mm:PinHeader_2x05_P2.54mm_Vertical, symbol Connector_Generic:Conn_02x05_Odd_Even
- added J24, J25, J26, J27, J28, J33: Conn_01x03_Male, Connector_PinHeader_2.54mm:PinHeader_1x03_P2.54mm_Vertical, symbol Connector:Conn_01x03_Male
- added R100, R19, R46, R73: 15K, Resistor_THT:R_Axial_DIN0204_L3.6mm_D1.6mm_P5.08mm_Horizontal, symbol Device:R
- added R15, R42, R69, R96: 100, Resistor_THT:R_Axial_DIN0204_L3.6mm_D1.6mm_P5.08mm_Horizontal, symbol Device:R
- C1, C2: renamed from C?; footprint (none) -> Capacitor_THT:CP_Radial_D5.0mm_P2.00mm
- C10, C13, C14, C15, C18, C19, C20, C23, C24, C25, C26, C27, C28, C29, C3, C30, C31, C32, C35, C4, C5, C8, C9: renamed from C?; footprint (none) -> Capacitor_SMD:C_0805_2012Metric_Pad1.18x1.45mm_HandSolder
- C11, C12, C16, C17, C21, C22, C6, C7: renamed from C?; footprint (none) -> Capacitor_THT:CP_Radial_D6.3mm_P2.50mm
- C33, C34: renamed from C?; footprint (none) -> Capacitor_THT:C_Radial_D10.0mm_H12.5mm_P5.00mm
- D1, D2, D3, D4: renamed from D?; footprint (none) -> Diode_THT:D_DO-15_P2.54mm_Vertical_KathodeUp
- J1, J10, J18, J4, J7: renamed from J?; footprint (none) -> Connector_PinSocket_2.54mm:PinSocket_1x03_P2.54mm_Vertical
- J11, J12, J2, J3, J5, J6, J8, J9: renamed from J?; footprint (none) -> Eurorack:AudioJack2_Tayda_A-2566
- J13: renamed from J?; value Bass -> Main Volume; footprint (none) -> Connector_PinSocket_2.54mm:PinSocket_1x06_P2.54mm_Vertical
- J14, J15, J16: renamed from J?; footprint (none) -> Connector_PinSocket_2.54mm:PinSocket_1x06_P2.54mm_Vertical
- J29, J30, J31, J32: renamed from J?; footprint (none) -> Connector_PinHeader_2.54mm:PinHeader_1x06_P2.54mm_Vertical
- J34: renamed from J?; footprint (none) -> Connector_PinHeader_2.54mm:PinHeader_1x03_P2.54mm_Vertical
- Q1, Q2, Q3, Q4, Q5, Q6, Q7, Q8: renamed from Q?; footprint (none) -> Package_TO_SOT_THT:TO-92_Inline_Wide
- Q10, Q11, Q12, Q9: renamed from Q?; footprint (none) -> Resistor_THT:R_Axial_DIN0204_L3.6mm_D1.6mm_P5.08mm_Horizontal
- R1, R10, R101, R102, R103, R104, R105, R106, R107, R108, R109, R11, R110, R111, R112, R113, R114, R115, R116, R117, R118, R119, R12, R120, R121, R122, R123, R124, R125, R126, R127, R128, R129, R13, R130, R131, R132, R133, R134, R135, R136, R137, R138, R139, R14, R140, R141, R142, R16, R17, R18, R2, R20, R21, R22, R23, R24, R25, R26, R27, R28, R29, R3, R30, R31, R32, R33, R34, R35, R36, R37, R38, R39, R4, R40, R41, R43, R44, R45, R47, R48, R49, R5, R50, R51, R52, R53, R54, R55, R56, R57, R58, R59, R6, R60, R61, R62, R63, R64, R65, R66, R67, R68, R7, R70, R71, R72, R74, R75, R76, R77, R78, R79, R8, R80, R81, R82, R83, R84, R85, R86, R87, R88, R89, R9, R90, R91, R92, R93, R94, R95, R97, R98, R99: renamed from R?; footprint (none) -> Resistor_THT:R_Axial_DIN0204_L3.6mm_D1.6mm_P5.08mm_Horizontal
- RV1, RV10, RV11, RV12, RV2, RV3, RV4, RV5, RV6, RV7, RV8, RV9: renamed from RV?; footprint (none) -> Eurorack:Potentiometer_RV16AF-41-15R1
- RV13: renamed from RV?; value 10K LOG -> 10K LOG x2; footprint (none) -> Eurorack:Potentiometer_RV16A01F-41-15R1
- RV14, RV15: renamed from RV?; value 100K LIN -> 100K LIN x2; footprint (none) -> Eurorack:Potentiometer_RV16A01F-41-15R1
- RV16: renamed from RV?; value 100K LOG -> 100K LOG x2; footprint (none) -> Eurorack:Potentiometer_RV16A01F-41-15R1
- U1, U10, U14, U15, U4, U7: renamed from U?; footprint (none) -> Package_DIP:DIP-14_W7.62mm_Socket
- U11, U2, U5, U8: renamed from U?; footprint (none) -> Package_SO:SOIC-16_3.9x9.9mm_P1.27mm
- U12, U13, U3, U6, U9: renamed from U?; footprint (none) -> Package_DIP:DIP-8_W7.62mm_Socket
- gave numbers to parts that had none: 5
Connections:
- net +12V: now also J24.3 (Pin_3), R100.1, R19.1, R46.1, R73.1
- net -12V: now also J24.1 (Pin_1)
- net GND: now also J22.2 (Pin_2), J23.3 (Pin_3), J23.4 (Pin_4), J23.5 (Pin_5), J23.6 (Pin_6), J23.7 (Pin_7), J23.8 (Pin_8), J24.2 (Pin_2), J33.2 (Pin_2), R15.1, R42.1, R69.1, R96.1
- net LVL_4': now also J28.1 (Pin_1)
- net at R140.2: now also J33.1 (Pin_1)
- net at R2.2: now also J22.1 (Pin_1)
- net at U8.14 (+): now also R69.2
- net at U8.15 (DIODE_BIAS): now also R73.2
- net at R1.2: now also J22.3 (Pin_3)
- net at U11.14 (+): now also R96.2
- net at U11.15 (DIODE_BIAS): now also R100.2
- net at U2.14 (+): now also R15.2
- net at U2.15 (DIODE_BIAS): now also R19.2
- net at R4.1: now also J23.1 (Pin_1), J23.2 (Pin_2)
- net at R3.1: now also J23.10 (Pin_10), J23.9 (Pin_9)
- net at U5.14 (+): now also R42.2
- net at U5.15 (DIODE_BIAS): now also R46.2
- net at R139.2: now also J33.3 (Pin_3)
- net CVP_1': no longer names the net of R6.1
- net CVP_1': now also J25.2 (Pin_2)
- net CVP_2': no longer names the net of R33.1
- net CVP_2': now also J26.2 (Pin_2)
- net CVP_3': no longer names the net of R60.1
- net CVP_3': now also J27.2 (Pin_2)
- net CVP_4': no longer names the net of R87.1
- net CVP_4': now also J28.2 (Pin_2)
- net LVL_1': no longer names the net of R12.2, U3.3 (+), U3.5 (+)
- net LVL_1': now also J25.1 (Pin_1)
- net LVL_2': no longer names the net of R39.2, U6.3 (+), U6.5 (+)
- net LVL_2': now also J26.1 (Pin_1)
- net LVL_3': no longer names the net of R66.2, U9.3 (+), U9.5 (+)
- net LVL_3': now also J27.1 (Pin_1)
- net PAN_1': no longer names the net of R5.1
- net PAN_1': now also J25.3 (Pin_3)
- net PAN_2': no longer names the net of R32.1
- net PAN_2': now also J26.3 (Pin_3)
- net PAN_3': no longer names the net of R59.1
- net PAN_3': now also J27.3 (Pin_3)
- net PAN_4': no longer names the net of R86.1
- net PAN_4': now also J28.3 (Pin_3)
- new net: J20.1 (Pin_1), J21.T
- new net: J19.S, J20.2 (Pin_2), J21.S
- new net: J19.T, J20.3 (Pin_3)
- no-connect marks 8 -> 10
Other:
- moved on the sheet: C1, C2, R3, R4

Commit message: pcbs populated
Parts:
- removed J17: AudioJack3, symbol Connector:AudioJack3
- removed J18: Conn_01x03_Female, Connector_PinSocket_2.54mm:PinSocket_1x03_P2.54mm_Vertical, symbol Connector:Conn_01x03_Female
- removed J32: Conn_01x06_Male, Connector_PinHeader_2.54mm:PinHeader_1x06_P2.54mm_Vertical, symbol Connector:Conn_01x06_Male
- added J30: >J16<, Connector_PinHeader_2.54mm:PinHeader_1x06_P2.54mm_Vertical, symbol Connector:Conn_01x06_Male
- added R143: 0, Resistor_THT:R_Axial_DIN0204_L3.6mm_D1.6mm_P1.90mm_Vertical, symbol Device:R
- H27: footprint Eurorack:Mech-AudioJack-Hole-0_25-L12B -> Eurorack:Mech-Potentiometer-Hole_level
- J21: renamed from J23; value Conn_02x05_Odd_Even -> RED LINE
- J22: renamed from J24; value Conn_01x03_Male -> >J20<
- J23: renamed from J25; value Conn_01x03_Male -> >J1<
- J24: renamed from J26; value Conn_01x03_Male -> >J4<
- J25: renamed from J27; value Conn_01x03_Male -> >J7<
- J26: renamed from J28; value Conn_01x03_Male -> >J10<
- J27: renamed from J29; value Conn_01x06_Male -> >J13<
- J28: renamed from J30; value Conn_01x06_Male -> >J15<
- J29: renamed from J31; value Conn_01x06_Male -> >J14<
- J31: renamed from J33; value Conn_01x03_Male -> >J18<
- J32: renamed from J34; value Conn_01x03_Male -> stereo_jack; footprint Connector_PinHeader_2.54mm:PinHeader_1x03_P2.54mm_Vertical -> Connector_Molex:Molex_KK-254_AE-6410-03A_1x03_P2.54mm_Vertical
- Q10, Q11, Q12, Q9: footprint Resistor_THT:R_Axial_DIN0204_L3.6mm_D1.6mm_P5.08mm_Horizontal -> Package_TO_SOT_THT:TO-92_Inline_Wide
- R1, R10, R100, R101, R102, R103, R104, R105, R106, R107, R108, R109, R11, R110, R111, R112, R113, R114, R115, R116, R117, R118, R119, R12, R120, R121, R122, R123, R124, R125, R126, R127, R128, R129, R13, R130, R131, R132, R133, R134, R135, R136, R137, R138, R139, R14, R140, R141, R142, R15, R16, R17, R18, R19, R2, R20, R21, R22, R23, R24, R25, R26, R27, R28, R29, R30, R31, R32, R33, R34, R35, R36, R37, R38, R39, R40, R41, R42, R43, R44, R45, R46, R47, R48, R49, R5, R50, R51, R52, R53, R54, R55, R56, R57, R58, R59, R6, R60, R61, R62, R63, R64, R65, R66, R67, R68, R69, R7, R70, R71, R72, R73, R74, R75, R76, R77, R78, R79, R8, R80, R81, R82, R83, R84, R85, R86, R87, R88, R89, R9, R90, R91, R92, R93, R94, R95, R96, R97, R98, R99: footprint Resistor_THT:R_Axial_DIN0204_L3.6mm_D1.6mm_P5.08mm_Horizontal -> Resistor_THT:R_Axial_DIN0204_L3.6mm_D1.6mm_P2.54mm_Vertical
- R3: renamed from R4; footprint Resistor_THT:R_Axial_DIN0204_L3.6mm_D1.6mm_P5.08mm_Horizontal -> Resistor_THT:R_Axial_DIN0204_L3.6mm_D1.6mm_P2.54mm_Vertical
- R4: renamed from R3; footprint Resistor_THT:R_Axial_DIN0204_L3.6mm_D1.6mm_P5.08mm_Horizontal -> Resistor_THT:R_Axial_DIN0204_L3.6mm_D1.6mm_P2.54mm_Vertical
- RV17, RV18, RV19, RV20: footprint (none) -> Eurorack:Potentiometer_Bourns_3362P_Vertical
- renumbered J19 to J17, J20 to J18, J21 to J19, J22 to J20
Connections:
- net GND: now also J30.3 (Pin_3), J30.6 (Pin_6); no longer J11.S, J12.S, J13.3 (Pin_3), J13.6 (Pin_6), J2.S, J20.2 (Pin_2), J3.S, J5.S, J6.S, J8.S, J9.S, RV11.1, RV12.1, RV13.3, RV13.6, RV2.1, RV3.1, RV5.1, RV6.1, RV8.1, RV9.1
- net at U15.3 (+): now also J30.5 (Pin_5)
- net at C34.2, R132.1: now also J30.4 (Pin_4)
- net at C33.2, R131.1: now also J30.1 (Pin_1)
- net at U15.5 (+): now also J30.2 (Pin_2)
- new net: J20.2 (Pin_2), R143.2
- new net GND': J11.S, J12.S, J13.3 (Pin_3), J13.6 (Pin_6), J2.S, J3.S, J5.S, J6.S, J8.S, J9.S, R143.1, RV11.1, RV12.1, RV13.3, RV13.6, RV2.1, RV3.1, RV5.1, RV6.1, RV8.1, RV9.1

Commit message: generated bom
Parts:
- removed J32: stereo_jack, Connector_Molex:Molex_KK-254_AE-6410-03A_1x03_P2.54mm_Vertical, symbol Connector:Conn_01x03_Male
- added H28, H29, H30, H31: MountingHole, Eurorack:Mech-MountingHole, symbol Mechanical:MountingHole
- added J32: AudioJack3, Eurorack:AudioJack3_Tayda_A-2585, symbol Connector:AudioJack3
- added J33: Conn_01x03_Female, Connector_PinSocket_2.54mm:PinSocket_1x03_P2.54mm_Vertical, symbol Connector:Conn_01x03_Female
- added J34: >J33<, Connector_PinHeader_2.54mm:PinHeader_1x03_P2.54mm_Vertical, symbol Connector:Conn_01x03_Male
- H16: value lvl4 -> lvl 4
- H24, H25: footprint Eurorack:Mech-AudioJack-Hole -> Eurorack:Mech-AudioJack-Hole-Output
- H26: footprint Eurorack:Mech-AudioJack-Hole-0_25-L12B -> Eurorack:Mech-AudioJack-Hole-Output
- Q1, Q2, Q3, Q4, Q5, Q6, Q7, Q8: value Q_PNP_CBE -> BC557B
- R1, R10, R100, R101, R102, R103, R104, R105, R106, R107, R108, R109, R11, R110, R111, R112, R113, R114, R115, R116, R117, R118, R119, R12, R120, R121, R122, R123, R124, R125, R126, R127, R128, R129, R13, R130, R131, R132, R133, R134, R135, R136, R137, R138, R139, R14, R140, R141, R142, R15, R16, R17, R18, R19, R2, R20, R21, R22, R23, R24, R25, R26, R27, R28, R29, R3, R30, R31, R32, R33, R34, R35, R36, R37, R38, R39, R4, R40, R41, R42, R43, R44, R45, R46, R47, R48, R49, R5, R50, R51, R52, R53, R54, R55, R56, R57, R58, R59, R6, R60, R61, R62, R63, R64, R65, R66, R67, R68, R69, R7, R70, R71, R72, R73, R74, R75, R76, R77, R78, R79, R8, R80, R81, R82, R83, R84, R85, R86, R87, R88, R89, R9, R90, R91, R92, R93, R94, R95, R96, R97, R98, R99: footprint Resistor_THT:R_Axial_DIN0204_L3.6mm_D1.6mm_P2.54mm_Vertical -> Eurorack:R_Axial_DIN0204_L3.6mm_D1.6mm_P2.54mm_Vertical
Connections:
- net GND: now also J34.1 (Pin_1)
- net GND': now also J17.S, J18.2 (Pin_2), J19.S, J32.S, J33.1 (Pin_1)
- net at R142.2: now also J34.3 (Pin_3)
- net at R141.2: now also J34.2 (Pin_2)
- new net: J32.R, J33.2 (Pin_2)
- new net: J32.T, J33.3 (Pin_3)
